Commit message: filter works?

File: src/deliberation/urdf/duckiebot.urdf (robot description, URDF)
Before this commit: robot duckiebot, 6 links, 5 joints
Links:
- link aarrgrpi/left_wheel_axis: geometry collision mesh filename=package://deliberation/urdf/duckiebot_leftwheel.dae; visual mesh filename=package://deliberation/urdf/duckiebot_leftwheel.dae
- link aarrgrpi/right_wheel_axis: geometry collision mesh filename=package://deliberation/urdf/duckiebot_rightwheel.dae; visual mesh filename=package://deliberation/urdf/duckiebot_rightwheel.dae
- link camera: geometry collision mesh filename=package://deliberation/urdf/duckiebot_camera.dae; visual mesh filename=package://deliberation/urdf/duckiebot_camera.dae
- link chassis: geometry collision mesh filename=package://deliberation/urdf/duckiebotFrame.dae; visual mesh filename=package://deliberation/urdf/duckiebotFrame.dae
- link computer: geometry collision mesh filename=package://deliberation/urdf/duckiebot_computer.dae; visual mesh filename=package://deliberation/urdf/duckiebot_computer.dae
